File: megaboard-01/megaboard-01.kicad_pcb (KiCad board)
At the start: 2 copper layers, 42.2 x 28.6 mm, 10 parts, among them J1 Conn_01x01_Pin, J2 Conn_01x01_Pin, J3 Conn_01x03_Pin, J4 Conn_01x01_Pin, J5 Conn_01x01_Pin, U1 THS3091DDAR

Commit message: change megaboard
Parts:
- added C2: C14663, Capacitor_SMD:C_0603_1608Metric, F.Cu at (189.7, 72.4)
- added C3: C1779, Capacitor_SMD:C_0805_2012Metric, F.Cu at (168.9, 112.4)
- added C4: C14663, Capacitor_SMD:C_0603_1608Metric, F.Cu at (184.6, 83.2)
- added C5: C57112, Capacitor_SMD:C_0603_1608Metric, F.Cu at (165.0, 112.4)
- added C6: C14663, Capacitor_SMD:C_0603_1608Metric, F.Cu at (192.9, 85.1)
- added J6: C37208, Connector_PinHeader_2.54mm:PinHeader_1x06_P2.54mm_Vertical, F.Cu at (165.3, 93.1)
- added J7: Conn_01x02_Pin, Connector_PinHeader_2.54mm:PinHeader_1x02_P2.54mm_Vertical, F.Cu at (214.0, 41.9)
- added J8: Conn_01x02_Pin, Connector_PinHeader_2.54mm:PinHeader_1x02_P2.54mm_Vertical, F.Cu at (207.0, 50.2)
- added R10: C17901, Resistor_SMD:R_1206_3216Metric, F.Cu at (160.2, 112.2)
- added R11: C17901, Resistor_SMD:R_1206_3216Metric, F.Cu at (160.2, 115.5)
- added R12: C17901, Resistor_SMD:R_1206_3216Metric, F.Cu at (160.2, 118.7)
- added R13: C17901, Resistor_SMD:R_1206_3216Metric, F.Cu at (160.2, 122.0)
- added R4: C17901, Resistor_SMD:R_1206_3216Metric, F.Cu at (160.2, 92.4)
- added R5: C17901, Resistor_SMD:R_1206_3216Metric, F.Cu at (160.2, 95.7)
- added R6: C17901, Resistor_SMD:R_1206_3216Metric, F.Cu at (160.2, 99.0)
- added R7: C17901, Resistor_SMD:R_1206_3216Metric, F.Cu at (160.2, 102.3)
- added R8: C17901, Resistor_SMD:R_1206_3216Metric, F.Cu at (160.2, 105.6)
- added R9: C17901, Resistor_SMD:R_1206_3216Metric, F.Cu at (160.2, 108.9)
- added T1: SWB1040-PCL, Mouser:SWB1040PCL, F.Cu at (231.8, 56.5)
- added U2: AD9833xRM, Package_SO:MSOP-10_3x3mm_P0.5mm, F.Cu at (200.5, 100.6)
- added X1: C558756, Crystal:Crystal_SMD_7050-4Pin_7.0x5.0mm, F.Cu at (178.0, 97.2)
- moved C1 23.8 mm to (125.6, 88.3)
- moved U1 23.8 mm to (120.5, 101.6)
- moved J1 23.8 mm to (120.8, 88.3)
- moved J2 23.8 mm to (130.8, 88.3)
- moved J4 23.8 mm to (107.3, 105.8)
- moved J5 23.8 mm to (130.8, 105.8)
- moved R1 23.8 mm to (102.5, 105.8)
- moved J3 23.8 mm to (107.3, 94.6)
- moved R2 23.8 mm to (111.8, 97.2)
- moved R3 23.8 mm to (132.1, 100.3)
Other:
- board text added: "FSYNC"
- board text added: "SCLK"
- board text added: "SDATA"
- board text added: "VCC"
- board text added: "VOUT"
