File: pcb/megaboard-01/megaboard-01.kicad_pcb (KiCad board)
At the start: 2 copper layers, 42.2 x 28.6 mm, 31 parts, among them J1 Conn_01x01_Pin, J2 Conn_01x01_Pin, J3 Conn_01x03_Pin, J4 Conn_01x01_Pin, J5 Conn_01x01_Pin, J6 C37208, J7 Conn_01x02_Pin, J8 Conn_01x02_Pin, T1 SWB1040-PCL, U1 THS3091DDAR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

Commit message: stuff
Parts:
- added C7: C116241, Capacitor_SMD:CP_Elec_8x10, F.Cu at (135.3, 101.9)
- added C8: C116241, Capacitor_SMD:CP_Elec_8x10, F.Cu at (135.3, 114.0)
- C1: value CC0603KRX7R9BB104 -> C14663
- J1, J2, J4, J5: value Conn_01x01_Pin -> C213184
- J3: value Conn_01x03_Pin -> C49257
- J7, J8: value Conn_01x02_Pin -> C492401
- R1: value RT0603BRE0750RL -> C849792
- R2: value 0603WAF1001T5E -> C21190
- R3: value RTT025002FTH -> C166559
- moved J7 101.2 mm to (167.1, 131.6), turned to -90 degrees
- moved T1 66.7 mm to (165.8, 66.1), turned to -90 degrees
- moved U2 57.4 mm to (145.2, 85.2), turned to 180 degrees
- moved C3 51.2 mm to (151.0, 64.4), turned to -90 degrees
- moved J4 45.0 mm to (149.2, 122.2)
- moved R1 44.4 mm to (143.7, 122.2)
- moved J8 44.2 mm to (164.5, 62.3), turned to -90 degrees
- moved C4 43.1 mm to (145.9, 64.4), turned to -90 degrees
- moved C6 41.8 mm to (151.3, 81.2), turned to 180 degrees
- moved C2 41.1 mm to (150.6, 85.0), turned to -90 degrees
- moved X1 35.8 mm to (148.7, 76.7), turned to 180 degrees
- moved R2 35.6 mm to (147.3, 94.9)
- moved U1 30.9 mm to (148.6, 114.6), turned to 90 degrees
- moved J6 28.7 mm to (150.6, 68.5), turned to -90 degrees
- moved C5 26.4 mm to (151.9, 89.4), turned to 180 degrees
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Routing:
- net Net-(J7-Pin_1): track 0.00 -> 89.4 mm
- net Net-(T1-SEC_2): track 0.00 -> 88.1 mm
- net Net-(J7-Pin_2): track 0.00 -> 64.2 mm
- net Net-(J6-Pin_1): track 0.00 -> 50.2 mm
- net Earth: track 16.6 -> 63.2 mm
- net GND1: track 0.00 -> 44.9 mm
- net Net-(J6-Pin_6): track 0.00 -> 20.4 mm
- net Net-(J6-Pin_5): track 0.00 -> 18.3 mm
- net Net-(J6-Pin_4): track 0.00 -> 17.6 mm
- net Net-(J6-Pin_3): track 0.00 -> 16.7 mm
- net Net-(U1--): track 27.7 -> 37.6 mm
- net Output: track 18.6 -> 10.3 mm
- net Net-(U2-MCLK): track 0.00 -> 6.74 mm
- net Input: track 15.9 -> 9.67 mm
- net -15V: track 35.0 -> 41.0 mm
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Other:
- board size 42.2 x 28.6 mm -> 50 x 76 mm
- board text added: "AD9833 BOARD"
- board text added: "AMPLIFICATION"
- board text added: "COUPLING"
- board text added: "LOAD IMPEDENCE"
- board text removed: "+15V"
- board text removed: "-15V"
- board text removed: "Coupling Cap"
- board text removed: "FSYNC"
- board text removed: "GND"
- board text removed: "Input"
- board text removed: "Output"
- board text removed: "SCLK"
- board text removed: "SDATA"
- board text removed: "VCC"
- board text removed: "VOUT"
