File: pcb/megaboard-01/megaboard-01.kicad_sch (KiCad schematic)
At the start: 31 parts, among them J1 Conn_01x01_Pin, J2 Conn_01x01_Pin, J3 Conn_01x03_Pin, J4 Conn_01x01_Pin, J5 Conn_01x01_Pin, J6 C37208, J7 Conn_01x02_Pin, J8 Conn_01x02_Pin, T1 SWB1040-PCL, U1 THS3091DDAR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

Commit message: stuff
Parts:
- added C7, C8: C116241, Capacitor_SMD:CP_Elec_8x10, symbol Device:C
Connections:
- net +15V: now also C7.1
- net -15V: now also C8.2
- net Earth: now also C7.2, C8.1
Other:
- note added: "AMPLIFICATION (RECOMMENDED CONFIGURATION FROM THS3091 + POWER STABILISATION)"
- note added: "C116241"
- note removed: "AMPLIFICATION (RECOMMENDED CONFIGURATION FROM THS3091)"
- moved on the sheet: C2, C3, C4, C5, C6, J3, J4, J5, J6, U2, X1

Commit message: stuff
Parts:
- C1: value CC0603KRX7R9BB104 -> C14663
- J1, J2, J4, J5: value Conn_01x01_Pin -> C213184
- J3: value Conn_01x03_Pin -> C49257
- J7, J8: value Conn_01x02_Pin -> C492401
- R1: value RT0603BRE0750RL -> C849792
- R2: value 0603WAF1001T5E -> C21190
- R3: value RTT025002FTH -> C166559
Changed lines of the file:
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@@
 			)
 		)
-		(property "Value" "Conn_01x01_Pin"
+		(property "Value" "C213184"
 			(at 179.705 39.37 0)
 			(effects
@@
 			)
 		)
-		(property "Value" "Conn_01x01_Pin"
+		(property "Value" "C213184"
 			(at 56.515 76.2 0)
 			(effects
@@
 			)
 		)
-		(property "Value" "Conn_01x03_Pin"
+		(property "Value" "C49257"
 			(at 26.035 45.72 0)
 			(effects
@@
 			)
 		)
-		(property "Value" "Conn_01x01_Pin"
+		(property "Value" "C213184"
 			(at 163.195 39.37 0)
 			(effects
@@
 			)
 		)
-		(property "Value" "RT0603BRE0750RL"
+		(property "Value" "C849792"
 			(at 97.79 41.9099 0)
 			(effects
@@
 			)
 		)
-		(property "Value" "RTT025002FTH"
+		(property "Value" "C166559"
 			(at 110.49 67.31 90)
 			(effects
@@
 			)
 		)
-		(property "Value" "CC0603KRX7R9BB104"
+		(property "Value" "C14663"
 			(at 171.45 36.83 90)
 			(effects
@@
 			)
 		)
-		(property "Value" "Conn_01x02_Pin"
+		(property "Value" "C492401"
 			(at 276.606 33.528 0)
 			(effects
@@
 			)
 		)
-		(property "Value" "Conn_01x01_Pin"
+		(property "Value" "C213184"
 			(at 56.515 85.09 0)
 			(effects
@@
 			)
 		)
-		(property "Value" "0603WAF1001T5E"
+		(property "Value" "C21190"
 			(at 87.63 67.31 90)
 			(effects
@@
 			)
 		)
-		(property "Value" "Conn_01x02_Pin"
+		(property "Value" "C492401"
 			(at 208.534 33.528 0)
 			(effects
